File: CH375_Serial.kicad_sch (KiCad schematic)
At the start: 36 parts, among them J1 USB_A, J2 DE9_Receptacle_MountingHoles, J3 Barrel_Jack_MountingPin, U1 CH375, U2 MAX3232, U3 IP4234CZ6, Y1 12MHz

Commit message: Added LCSC part numbers for most, exported simple BOM
Parts:
- C1, C13, C2, C3, C4, C5, C6, C7: LCSC (none) -> C49678
- C10: LCSC (none) -> C13967
- C11, C12: LCSC (none) -> C340733
- C8, C9: LCSC (none) -> C1798
- D1, F1: now left out of the parts list
- FB1: LCSC (none) -> C1015
- J1: LCSC (none) -> C456018
- J2: LCSC (none) -> C19077337
- J3: LCSC (none) -> C16214
- R1: LCSC (none) -> C17513
- R3: LCSC (none) -> C17673
- U1: LCSC (none) -> C8962
- U2: LCSC (none) -> C193666
- U3: LCSC (none) -> C355086
- Y1: LCSC (none) -> C2857630
